Commit message: new cast_urdf

File: urdf/cast_wt_auxTable.urdf (robot description, URDF)
Before this commit: robot cast_flying_arena, 3 links, 2 joints
Links:
- removed link wind_tunnel
- added link windtunnel; visual mesh filename=package://bintel_ros/meshes/wind_tunnel_down.dae
Joints:
- removed joint world_to_auxTable
- removed joint world_to_wind_tunnel
- added joint j1: type fixed, parent world, child auxTable, origin xyz=0.0 0.0 2 rpy=0 0 0
- added joint j2: type fixed, parent world, child windtunnel, origin xyz=0 -7.7 0 rpy=0 0 1.5707

File: urdf/inteldrone_2.urdf (robot description, URDF)
Before this commit: robot intelaero, 7 links, 4 joints
Links:
- removed link r200lidar
- added link base_link
- added link camera_link; visual mesh filename=package://bintel_ros/meshes/r200.STL scale=0.001 0.001 0.001
Joints:
- added joint bintel_t0_engineLL: type fixed, parent bintel, child engineLL, origin xyz=0.128 -0.128 0.02 rpy=0 0 3.1415
- added joint bintel_t0_engineLR: type fixed, parent bintel, child engineLR, origin xyz=0.128 0.128 0.02 rpy=0 0 3.1415
- added joint bintel_to_base_link: type fixed, parent bintel, child base_link, origin xyz=0 0 0 rpy=0 0 0
- joint bintel_t0_engineUL: origin xyz=0.125 -0.125 0.02 rpy=0 0 3.1415 -> xyz=-0.128 -0.128 0.02 rpy=0 0 3.1415
- joint bintel_t0_engineUR: origin xyz=0.125 0.125 0.02 rpy=0 0 3.1415 -> xyz=-0.128 0.128 0.02 rpy=0 0 3.1415
- joint laser_to_bintel: origin xyz=0.03 0.0 0.05 rpy=0 0 3.1415 -> xyz=0.03 0.0 0.07 rpy=0 0 3.1415
- joint lidar_bintel: child r200lidar -> camera_link; origin xyz=-0.11 0.0 -0.01 rpy=0 0 3.1415 -> xyz=-0.11 0.0 -0.014 rpy=0 0 3.141592
