Commit message: Added new intel down and intel USC urdfs

File: urdf/inteldrone_USC.urdf (robot description, URDF)
Before this commit: robot intelaero, 10 links, 9 joints
Links:
- removed link bintel
- added link intel_drone; visual mesh filename=package://bintel_ros/meshes/inteldrone_frame.stl scale=0.001 0.001 0.001
Joints:
- removed joint bintel_t0_engineLL
- removed joint bintel_t0_engineLR
- removed joint bintel_t0_engineUL
- removed joint bintel_t0_engineUR
- removed joint bintel_to_base_link
- removed joint laser_to_bintel
- removed joint lidar_bintel
- added joint intel_drone_t0_engineLL: type fixed, parent intel_drone, child engineLL, origin xyz=0.128 -0.128 0.02 rpy=0 0 3.1415
- added joint intel_drone_t0_engineLR: type fixed, parent intel_drone, child engineLR, origin xyz=0.128 0.128 0.02 rpy=0 0 3.1415
- added joint intel_drone_t0_engineUL: type fixed, parent intel_drone, child engineUL, origin xyz=-0.128 -0.128 0.02 rpy=0 0 3.1415
- added joint intel_drone_t0_engineUR: type fixed, parent intel_drone, child engineUR, origin xyz=-0.128 0.128 0.02 rpy=0 0 3.1415
- added joint intel_drone_to_base_link: type fixed, parent intel_drone, child base_link, origin xyz=0 0 0 rpy=0 0 0
- added joint laser_to_intel_drone: type fixed, parent intel_drone, child laser, origin xyz=0.05 0.0 0.05 rpy=0 0 0
- added joint lidar_intel_drone: type fixed, parent intel_drone, child camera_link, origin xyz=0.11 0.0 -0.014 rpy=0 0 0

File: urdf/inteldrone_down.urdf (robot description, URDF)
Before this commit: robot intelaero, 10 links, 9 joints
Joints:
- joint camera_depth: origin xyz=0.0 0.0 0.0 rpy=0 0 0 -> xyz=0.0 0.0 0.0 rpy=1.5707 0 0
