Commit message: rehearsal for ISER working

File: urdf/inteldrone_down.urdf (robot description, URDF)
Before this commit: robot intelaero, 10 links, 9 joints
Joints:
- joint laser_to_bintel: origin xyz=0.03 0.0 0.07 rpy=0 0 3.1415 -> xyz=0.03 0.0 0.07 rpy=0 0 0
- joint lidar_bintel: origin xyz=-0.11 0.0 -0.014 rpy=0 1.5707 3.141592 -> xyz=0.11 0.0 -0.014 rpy=0 1.5707 3.141592

Commit message: add save bag file LTF and increase rates

File: urdf/inteldrone_down.urdf (robot description, URDF)
Before this commit: robot intelaero, 10 links, 9 joints
Joints:
- joint camera_depth: origin xyz=0.0 0.0 0.0 rpy=1.5707 0 0 -> xyz=0.0 0.0 0.0 rpy=0 0 0
- joint lidar_bintel: origin xyz=0.11 0.0 -0.014 rpy=0 1.5707 3.141592 -> xyz=0.11 0.0 -0.014 rpy=0 1.57 0
