Commit message: change vrpn launch

File: urdf/cast.urdf (robot description, URDF)
Before this commit: robot cast_flying_arena, 1 links, 0 joints
Links:
- removed link world
- added link map; visual mesh filename=package://bintel_ros/meshes/cast/cast_simple_2.dae

Commit message: urdf cast changed

File: urdf/cast.urdf (robot description, URDF)
Before this commit: robot cast_flying_arena, 1 links, 0 joints
Links:
- removed link map
- added link world; visual mesh filename=package://bintel_ros/meshes/cast/cast_simple_2.dae
